File: kicad/pcb/board.kicad_pcb (KiCad board)
At the start: 0 parts

Commit message: Signed-off-by: Dmitry Ponyatov <dponyatov@samsa.local>
Other:
- copper layers 0 -> 2
Changed lines of the file:
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@@
 (kicad_pcb (version 20211014) (generator pcbnew)
+  (general
+    (thickness 1.6)
+  )
+  (paper "A4")
+  (layers
+    (0 "F.Cu" signal)
+    (31 "B.Cu" signal)
+    (44 "Edge.Cuts" user)
+  )
 )
